File: hardware/proteus-br/lowside_quad.kicad_sch (KiCad schematic)
At the start: 12 parts, among them U301 VNLD5160, U302 VNLD5160

Commit message: proteus-br: title blocks v1 + PWR_FLAG no VDDA (mcu/psu/lowside atualizados)
Parts:
- removed RN301, RN302: 1k, Resistor_SMD:R_Array_Convex_4x0603, symbol Device:R_Pack04
- U301, U302: LCSC N/A -> C377942; MFN (none) -> STMicroelectronics; MPN (none) -> VNLD5160TR-E
Other:
- company: rusEFI -> baseado em rusEFI Proteus v0.7
- title: rusEfi Proteus -> Proteus-BR — lowside_quad
Changed lines of the file:
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@@
   (paper "A4")
   (title_block
-    (title "rusEfi Proteus")
-    (date "2022-04-09")
-    (rev "v0.7")
-    (company "rusEFI")
+    (title "Proteus-BR — lowside_quad")
+    (date "2026-06-11")
+    (rev "v1")
+    (company "baseado em rusEFI Proteus v0.7")
     (comment 1 "github.com/mck1117/proteus")
     (comment 2 "rusefi.com/s/proteus")
@@
     (property "Datasheet" "~" (at 108.585 57.785 0) (effects (font (size 1.524 1.524)) hide))
     (property "PN" "VNLD5160TR-E" (at 106.045 51.435 0) (effects (font (size 1.27 1.27)) hide))
-    (property "LCSC" "N/A" (at 106.045 51.435 0) (effects (font (size 1.27 1.27)) hide))
+    (property "LCSC" "C377942" (at 106.045 51.435 0) (effects (font (size 1.27 1.27)) hide))
+    (property "MFN" "STMicroelectronics" (at 106.045 35.0012 0) (effects (font (size 1.27 1.27)) hide))
+    (property "MPN" "VNLD5160TR-E" (at 106.045 35.0012 0) (effects (font (size 1.27 1.27)) hide))
     (pin "1")
     (pin "2")
@@
     (property "Datasheet" "~" (at 108.585 99.695 0) (effects (font (size 1.524 1.524)) hide))
     (property "PN" "VNLD5160TR-E" (at 106.045 93.345 0) (effects (font (size 1.27 1.27)) hide))
-    (property "LCSC" "N/A" (at 106.045 93.345 0) (effects (font (size 1.27 1.27)) hide))
+    (property "LCSC" "C377942" (at 106.045 93.345 0) (effects (font (size 1.27 1.27)) hide))
+    (property "MFN" "STMicroelectronics" (at 106.045 76.9112 0) (effects (font (size 1.27 1.27)) hide))
+    (property "MPN" "VNLD5160TR-E" (at 106.045 76.9112 0) (effects (font (size 1.27 1.27)) hide))
     (pin "1")
     (pin "2")
@@
           (unit 1)
         )
-      )
-    )
-  )
-  (symbol
-    (lib_id "Device:R_Pack04")
-    (at 78.105 71.12 270)
-    (mirror x)
-    (unit 1)
-    (in_bom yes)
-    (on_board yes)
-    (dnp no)
-    (property "Reference" "RN301" (at 78.105 81.7118 90) (effects (font (size 1.27 1.27))))
-    (property "Value" "1k" (at 78.105 79.4004 90) (effects (font (size 1.27 1.27))))
-    (property "Footprint" "Resistor_SMD:R_Array_Convex_4x0603"
-      (at 78.105 64.135 90)
-      (effects (font (size 1.27 1.27)) hide)
-    )
-    (property "Datasheet" "~" (at 78.105 71.12 0) (effects (font (size 1.27 1.27)) hide))
-    (property "PN" "" (at 78.105 71.12 0) (effects (font (size 1.27 1.27)) hide))
-    (property "LCSC" "C20197" (at 78.105 71.12 0) (effects (font (size 1.27 1.27)) hide))
-    (property "LCSC_ext" "0" (at 78.105 71.12 0) (effects (font (size 1.27 1.27)) hide))
-    (pin "1")
-    (pin "2")
-    (pin "3")
-    (pin "4")
-    (pin "5")
-    (pin "6")
-    (pin "7")
-    (pin "8")
-    (instances
-      (project "proteus-br"
-        (path "/da96cc1d-20c0-47ba-9881-2a73783a20fb/00000000-0000-0000-0000-00005d99f107"
-          (reference "RN301")
-          (unit 1)
-        )
-        (path "/da96cc1d-20c0-47ba-9881-2a73783a20fb/00000000-0000-0000-0000-00005d99f54c"
-          (reference "RN501")
-          (unit 1)
-        )
-        (path "/da96cc1d-20c0-47ba-9881-2a73783a20fb/00000000-0000-0000-0000-00005d98a146"
-          (reference "RN201")
-          (unit 1)
-        )
-        (path "/da96cc1d-20c0-47ba-9881-2a73783a20fb/00000000-0000-0000-0000-00005d99f37f"
-          (reference "RN401")
-          (unit 1)
-        )
-      )
-    )
-  )
-  (symbol
-    (lib_id "Device:R_Pack04")
-    (at 67.945 83.82 0)
-    (unit 1)
-    (in_bom yes)
-    (on_board yes)
-    (dnp no)
-    (property "Reference" "RN302" (at 57.3532 83.82 90) (effects (font (size 1.27 1.27))))
-    (property "Value" "1k" (at 59.6646 83.82 90) (effects (font (size 1.27 1.27))))
-    (property "Footprint" "Resistor_SMD:R_Array_Convex_4x0603"
-      (at 74.93 83.82 90)
-      (effects (font (size 1.27 1.27)) hide)
-    )
-    (property "Datasheet" "~" (at 67.945 83.82 0) (effects (font (size 1.27 1.27)) hide))
-    (property "PN" "" (at 67.945 83.82 0) (effects (font (size 1.27 1.27)) hide))
-    (property "LCSC" "C20197" (at 67.945 83.82 0) (effects (font (size 1.27 1.27)) hide))
-    (property "LCSC_ext" "0" (at 67.945 83.82 0) (effects (font (size 1.27 1.27)) hide))
-    (pin "1")
-    (pin "2")
-    (pin "3")
-    (pin "4")
-    (pin "5")
-    (pin "6")
-    (pin "7")
-    (pin "8")
-    (instances
-      (project "proteus-br"
-        (path "/da96cc1d-20c0-47ba-9881-2a73783a20fb/00000000-0000-0000-0000-00005d99f107"
-          (reference "RN302")
-          (unit 1)
-        )
-        (path "/da96cc1d-20c0-47ba-9881-2a73783a20fb/00000000-0000-0000-0000-00005d99f54c"
-          (reference "RN502")
-          (unit 1)
-        )
-        (path "/da96cc1d-20c0-47ba-9881-2a73783a20fb/00000000-0000-0000-0000-00005d98a146"
-          (reference "RN202")
-          (unit 1)
-        )
-        (path "/da96cc1d-20c0-47ba-9881-2a73783a20fb/00000000-0000-0000-0000-00005d99f37f"
-          (reference "RN402")
-          (unit 1)
-        )
