File: hardware/proteus-br/psu.kicad_sch (KiCad schematic)
At the start: 33 parts, among them U1004 TLE4251D, U1005 TLE4251D, U6 TJA1051T-3, U902 AMS1117-3.3, U903 LMR14020, U904 TJA1051T-3

Commit message: proteus-br: title blocks v1 + PWR_FLAG no VDDA (mcu/psu/lowside atualizados)
Parts:
- C905: footprint Capacitor_SMD:C_0402_1005Metric -> Capacitor_SMD:C_0603_1608Metric
- D1, D2: MFN (none) -> Nexperia; MPN (none) -> PESD1CAN,215
- D1001: LCSC C151281 -> C133707; MFN (none) -> STMicroelectronics; MPN (none) -> SM15T33CA
- R1006, R1007, R905, R906, R907, R908: footprint Resistor_SMD:R_0402_1005Metric -> Resistor_SMD:R_0603_1608Metric
- U1004, U1005: LCSC N/A -> C539669; MFN (none) -> Infineon; MPN (none) -> TLE4251D
- U6, U904: MFN (none) -> NXP; MPN (none) -> TJA1051T/3
- U902: MFN (none) -> AMS; MPN (none) -> AMS1117-3.3
- U903: MFN (none) -> Texas Instruments; MPN (none) -> LMR14020SDDAR
Other:
- company: rusEFI -> baseado em rusEFI Proteus v0.7
- title: rusEfi Proteus -> Proteus-BR — psu
Changed lines of the file:
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@@
   (paper "A4")
   (title_block
-    (title "rusEfi Proteus")
-    (date "2022-04-09")
-    (rev "v0.7")
-    (company "rusEFI")
+    (title "Proteus-BR — psu")
+    (date "2026-06-11")
+    (rev "v1")
+    (company "baseado em rusEFI Proteus v0.7")
     (comment 1 "github.com/mck1117/proteus")
     (comment 2 "rusefi.com/s/proteus")
@@
     (property "Datasheet" "~" (at 31.75 34.29 0) (effects (font (size 1.27 1.27)) hide))
     (property "PN" "SM15T33CA" (at 31.75 34.29 0) (effects (font (size 1.27 1.27)) hide))
-    (property "LCSC" "C151281" (at 31.75 34.29 0) (effects (font (size 1.27 1.27)) hide))
+    (property "LCSC" "C133707" (at 31.75 34.29 0) (effects (font (size 1.27 1.27)) hide))
     (property "LCSC_ext" "1" (at 31.75 34.29 0) (effects (font (size 1.27 1.27)) hide))
     (property "possible_not_ext" "1" (at 31.75 34.29 0) (effects (font (size 1.27 1.27)) hide))
+    (property "MFN" "STMicroelectronics" (at 33.7566 33.1216 0) (effects (font (size 1.27 1.27)) hide))
+    (property "MPN" "SM15T33CA" (at 33.7566 33.1216 0) (effects (font (size 1.27 1.27)) hide))
     (pin "1")
     (pin "2")
@@
     (property "Datasheet" "~" (at 44.45 78.105 0) (effects (font (size 1.27 1.27)) hide))
     (property "PN" "TLS115D0E" (at 44.45 78.105 0) (effects (font (size 1.27 1.27)) hide))
-    (property "LCSC" "N/A" (at 44.45 78.105 0) (effects (font (size 1.27 1.27)) hide))
+    (property "LCSC" "C539669" (at 44.45 78.105 0) (effects (font (size 1.27 1.27)) hide))
+    (property "MFN" "Infineon" (at 45.085 69.85 0) (effects (font (size 1.27 1.27)) hide))
+    (property "MPN" "TLE4251D" (at 45.085 69.85 0) (effects (font (size 1.27 1.27)) hide))
     (pin "1")
     (pin "2")
@@
     (property "Reference" "R1006" (at 54.61 94.4372 90) (effects (font (size 1.27 1.27))))
     (property "Value" "10k" (at 54.61 96.7486 90) (effects (font (size 1.27 1.27))))
-    (property "Footprint" "Resistor_SMD:R_0402_1005Metric"
+    (property "Footprint" "Resistor_SMD:R_0603_1608Metric"
       (at 54.61 97.917 90)
       (effects (font (size 1.27 1.27)) hide)
@@
     (property "Datasheet" "~" (at 117.475 78.105 0) (effects (font (size 1.27 1.27)) hide))
     (property "PN" "TLS115D0E" (at 117.475 78.105 0) (effects (font (size 1.27 1.27)) hide))
-    (property "LCSC" "N/A" (at 117.475 78.105 0) (effects (font (size 1.27 1.27)) hide))
+    (property "LCSC" "C539669" (at 117.475 78.105 0) (effects (font (size 1.27 1.27)) hide))
     (property "DNP" "DNP fase 1" (at 118.11 69.85 0) (effects (font (size 1.27 1.27)) hide))
+    (property "MFN" "Infineon" (at 118.11 69.85 0) (effects (font (size 1.27 1.27)) hide))
+    (property "MPN" "TLE4251D" (at 118.11 69.85 0) (effects (font (size 1.27 1.27)) hide))
     (pin "1")
     (pin "2")
@@
     (property "Reference" "R1007" (at 127.635 94.4372 90) (effects (font (size 1.27 1.27))))
     (property "Value" "10k" (at 127.635 96.7486 90) (effects (font (size 1.27 1.27))))
-    (property "Footprint" "Resistor_SMD:R_0402_1005Metric"
+    (property "Footprint" "Resistor_SMD:R_0603_1608Metric"
       (at 127.635 97.917 90)
       (effects (font (size 1.27 1.27)) hide)
@@
     (property "LCSC" "C152727" (at 227.33 81.915 0) (effects (font (size 1.27 1.27)) hide))
     (property "LCSC_ext" "1" (at 227.33 81.915 0) (effects (font (size 1.27 1.27)) hide))
+    (property "MFN" "Nexperia" (at 225.3488 83.0834 0) (effects (font (size 1.27 1.27)) hide))
+    (property "MPN" "PESD1CAN,215" (at 225.3488 83.0834 0) (effects (font (size 1.27 1.27)) hide))
     (pin "1")
     (pin "2")
@@
     (property "Reference" "R906" (at 89.408 33.7566 0) (effects (font (size 1.27 1.27)) (justify left)))
     (property "Value" "1" (at 89.408 36.068 0) (effects (font (size 1.27 1.27)) (justify left)))
-    (property "Footprint" "Resistor_SMD:R_0402_1005Metric"
+    (property "Footprint" "Resistor_SMD:R_0603_1608Metric"
       (at 85.852 34.925 90)
       (effects (font (size 1.27 1.27)) hide)
@@
     (property "PN" "LMR14020" (at 137.16 34.29 0) (effects (font (size 1.27 1.27)) hide))
     (property "possible_not_ext" "0" (at 137.16 34.29 0) (effects (font (size 1.27 1.27)) hide))
+    (property "MFN" "Texas Instruments" (at 139.7 23.495 0) (effects (font (size 1.27 1.27)) hide))
+    (property "MPN" "LMR14020SDDAR" (at 139.7 23.495 0) (effects (font (size 1.27 1.27)) hide))
     (pin "1")
     (pin "2")
@@
     (property "Reference" "R908" (at 158.75 39.37 90) (effects (font (size 1.27 1.27))))
     (property "Value" "68k" (at 158.75 41.91 90) (effects (font (size 1.27 1.27))))
-    (property "Footprint" "Resistor_SMD:R_0402_1005Metric"
+    (property "Footprint" "Resistor_SMD:R_0603_1608Metric"
       (at 158.75 43.688 90)
       (effects (font (size 1.27 1.27)) hide)
@@
     (property "Reference" "R907" (at 149.86 51.435 90) (effects (font (size 1.27 1.27)) (justify left)))
     (property "Value" "12k" (at 152.4 50.8 90) (effects (font (size 1.27 1.27)) (justify left)))
-    (property "Footprint" "Resistor_SMD:R_0402_1005Metric"
+    (property "Footprint" "Resistor_SMD:R_0603_1608Metric"
       (at 150.622 48.895 90)
       (effects (font (size 1.27 1.27)) hide)
@@
     (property "Reference" "C905" (at 162.56 43.815 90) (effects (font (size 1.27 1.27))))
     (property "Value" "330p" (at 162.56 50.165 90) (effects (font (size 1.27 1.27))))
-    (property "Footprint" "Capacitor_SMD:C_0402_1005Metric"
+    (property "Footprint" "Capacitor_SMD:C_0603_1608Metric"
       (at 158.75 47.9552 0)
       (effects (font (size 1.27 1.27)) hide)
@@
     )
     (property "Value" "10k" (at 119.888 44.323 0) (effects (font (size 1.27 1.27)) (justify left)))
-    (property "Footprint" "Resistor_SMD:R_0402_1005Metric"
+    (property "Footprint" "Resistor_SMD:R_0603_1608Metric"
       (at 116.332 43.18 90)
       (effects (font (size 1.27 1.27)) hide)
@@
     (property "LCSC" "C38695" (at 190.5 81.915 0) (effects (font (size 1.27 1.27)) hide))
     (property "LCSC_ext" "0" (at 190.5 81.915 0) (effects (font (size 1.27 1.27)) hide))
+    (property "MFN" "NXP" (at 181.61 90.805 0) (effects (font (size 1.27 1.27)) hide))
+    (property "MPN" "TJA1051T/3" (at 181.61 90.805 0) (effects (font (size 1.27 1.27)) hide))
     (pin "1")
     (pin "2")
@@
     (property "LCSC" "C6186" (at 222.25 29.21 0) (effects (font (size 1.27 1.27)) hide))
     (property "LCSC_ext" "0" (at 222.25 29.21 0) (effects (font (size 1.27 1.27)) hide))
+    (property "MFN" "AMS" (at 222.25 23.0632 0) (effects (font (size 1.27 1.27)) hide))
+    (property "MPN" "AMS1117-3.3" (at 222.25 23.0632 0) (effects (font (size 1.27 1.27)) hide))
     (pin "1")
     (pin "2")
@@
       (effects (font (size 1.27 1.27)) hide)
     )
+    (property "MFN" "Nexperia" (at 225.3488 126.2634 0) (effects (font (size 1.27 1.27)) hide))
+    (property "MPN" "PESD1CAN,215" (at 225.3488 126.2634 0) (effects (font (size 1.27 1.27)) hide))
     (pin "1")
     (pin "2")
@@
       (effects (font (size 1.27 1.27)) hide)
     )
-    (pin "1")
-    (pin "2")
+    (property "MFN" "NXP" (at 181.61 133.985 0) (effects (font (size 1.27 1.27)) hide))
+    (property "MPN" "TJA1051T/3" (at 181.61 133.985 0) (effects (font (size 1.27 1.27)) hide))
+    (pin "1")
+    (pin "2")
